File: cnc-universal-input.sch (KiCad schematic (older format))
At the start: 155 parts, among them J1 SA, J10 pwr-in, J11 output, J12 USB_B_Mini, J13 ext-pwr, J2 SB, J3 SC, J4 SD, J5 SE, J6 SF, J7 SG, J8 SH, J9 AVR-ISP-6, Q1 2N7002, Q10 IRLML2244TRPBF, Q2 2N7002, Q3 2N7002, Q4 2N7002, Q5 2N7002, Q6 2N7002, Q7 2N7002, Q8 2N7002, Q9 2N7002, SW1 RESET, SW2 BTN, U1 ATmega328P, U10 SFH617A-4, U11 SFH617A-4, U12 SFH617A-4, U13 SFH617A-4, U14 SFH617A-4, U15 SFH617A-4, U16 SFH617A-4, U17 SFH617A-4, U18 CH340G, U2 74HC595, U3 74HC595, U4 74HC595, U5 4051, U6 L7812, U7 L7805, U8 LM7321, U9 SFH617A-4, Y1 20Mhz, Y2 12MHz

Commit message: 4051s suck
4051s exist as HC version... did you know that?
Parts:
- added Q11, Q12, Q13: 2N7002, Package_TO_SOT_SMD:SOT-23, symbol Transistor_FET:2N7002
- added R69, R70, R71: 10K, Resistor_SMD:R_0805_2012Metric, symbol Device:R_Small
- U1: value ATmega328P -> ATmega328PB
Connections:
- net labels added: SSELAH, SSELBH, SSELCH
- wire segments 562 -> 586
Changed lines of the file:
@@
 P 10550 6200
 F 0 "U1" H 10900 7700 50  0000 C CNN
-F 1 "ATmega328P" V 10500 6300 50  0000 C CNN
+F 1 "ATmega328PB" V 10500 6300 50  0000 C CNN
 F 2 "Package_QFP:TQFP-32_7x7mm_P0.8mm" H 10550 6200 50  0001 C CIN
 F 3 "http://ww1.microchip.com/downloads/en/DeviceDoc/ATmega328_P%20AVR%20MCU%20with%20picoPower%20Technology%20Data%20Sheet%2040001984A.pdf" H 10550 6200 50  0001 C CNN
@@
 	1    0    0    -1
 $EndComp
-Text Label 11800 2200 2    50   ~ 0
+Text Label 11950 3850 2    50   ~ 0
 SSELA
-Text Label 11800 2300 2    50   ~ 0
-SSELB
-Text Label 11800 2400 2    50   ~ 0
-SSELC
 Wire Notes Line
 	6200 550  6200 2850
@@
 ASIN
 Wire Notes Line
-	14100 3100 11350 3100
+	14100 4000 11350 4000
 Wire Notes Line
-	11350 3100 11350 550
+	11350 4000 11350 550
 Wire Notes Line
 	11350 550  14100 550
 Wire Notes Line
-	14100 550  14100 3100
+	14100 550  14100 4000
 Text Notes 11300 2050 1    79   ~ 0
 SENSE
@@
 	1    0    0    -1
 $EndComp
+$Comp
+L Transistor_FET:2N7002 Q11
+U 1 1 6009DBE7
+P 12050 3650
+F 0 "Q11" V 11950 3550 50  0000 C CNN
+F 1 "2N7002" V 11950 3950 50  0000 C CNN
+F 2 "Package_TO_SOT_SMD:SOT-23" H 12250 3575 50  0001 L CIN
+F 3 "https://www.fairchildsemi.com/datasheets/2N/2N7002.pdf" H 12050 3650 50  0001 L CNN
+	1    12050 3650
+	0    -1   -1   0
+$EndComp
+$Comp
+L Device:R_Small R69
+U 1 1 600A062B
+P 11700 3550
+F 0 "R69" V 11600 3500 50  0000 L CNN
+F 1 "10K" V 11800 3450 50  0000 L CNN
+F 2 "Resistor_SMD:R_0805_2012Metric" H 11700 3550 50  0001 C CNN
+F 3 "~" H 11700 3550 50  0001 C CNN
+	1    11700 3550
+	0    -1   -1   0
+$EndComp
+Wire Wire Line
+	11800 3550 11850 3550
+$Comp
+L power:+12V #PWR0206
+U 1 1 600FB559
+P 11550 3500
+F 0 "#PWR0206" H 11550 3350 50  0001 C CNN
+F 1 "+12V" H 11565 3673 50  0000 C CNN
+F 2 "" H 11550 3500 50  0001 C CNN
+F 3 "" H 11550 3500 50  0001 C CNN
+	1    11550 3500
+	1    0    0    -1
+$EndComp
+Wire Wire Line
+	11950 3850 12050 3850
+Text Label 12000 3400 0    50   ~ 0
+SSELAH
+Wire Wire Line
+	12300 3650 12300 3550
+Wire Wire Line
+	12300 3550 12250 3550
+Text Label 11800 2200 2    50   ~ 0
+SSELAH
+Text Label 11800 2300 2    50   ~ 0
+SSELBH
+Text Label 11800 2400 2    50   ~ 0
+SSELCH
+Connection ~ 11800 3550
+Wire Wire Line
+	11550 3500 11550 3550
+Wire Wire Line
+	11550 3550 11600 3550
+Wire Wire Line
+	11800 3400 12000 3400
+Wire Wire Line
+	11800 3400 11800 3550
+$Comp
+L power:GND #PWR0207
+U 1 1 605ACDEE
+P 12300 3650
+F 0 "#PWR0207" H 12300 3400 50  0001 C CNN
+F 1 "GND" H 12305 3477 50  0000 C CNN
+F 2 "" H 12300 3650 50  0001 C CNN
+F 3 "" H 12300 3650 50  0001 C CNN
+	1    12300 3650
+	1    0    0    -1
+$EndComp
+Text Label 12800 3850 2    50   ~ 0
+SSELB
+$Comp
+L Transistor_FET:2N7002 Q12
+U 1 1 60669982
+P 12900 3650
+F 0 "Q12" V 12800 3550 50  0000 C CNN
+F 1 "2N7002" V 12800 3950 50  0000 C CNN
+F 2 "Package_TO_SOT_SMD:SOT-23" H 13100 3575 50  0001 L CIN
+F 3 "https://www.fairchildsemi.com/datasheets/2N/2N7002.pdf" H 12900 3650 50  0001 L CNN
+	1    12900 3650
+	0    -1   -1   0
+$EndComp
+$Comp
+L Device:R_Small R70
+U 1 1 60669988
+P 12550 3550
+F 0 "R70" V 12450 3500 50  0000 L CNN
+F 1 "10K" V 12650 3450 50  0000 L CNN
+F 2 "Resistor_SMD:R_0805_2012Metric" H 12550 3550 50  0001 C CNN
+F 3 "~" H 12550 3550 50  0001 C CNN
+	1    12550 3550
+	0    -1   -1   0
+$EndComp
+Wire Wire Line
+	12650 3550 12700 3550
+$Comp
+L power:+12V #PWR0208
+U 1 1 6066998F
+P 12400 3500
+F 0 "#PWR0208" H 12400 3350 50  0001 C CNN
+F 1 "+12V" H 12415 3673 50  0000 C CNN
+F 2 "" H 12400 3500 50  0001 C CNN
+F 3 "" H 12400 3500 50  0001 C CNN
+	1    12400 3500
+	1    0    0    -1
+$EndComp
+Wire Wire Line
+	12800 3850 12900 3850
+Text Label 12850 3400 0    50   ~ 0
+SSELBH
+Wire Wire Line
+	13150 3650 13150 3550
+Wire Wire Line
+	13150 3550 13100 3550
+Connection ~ 12650 3550
+Wire Wire Line
+	12400 3500 12400 3550
+Wire Wire Line
+	12400 3550 12450 3550
+Wire Wire Line
+	12650 3400 12850 3400
+Wire Wire Line
+	12650 3400 12650 3550
+$Comp
+L power:GND #PWR0209
+U 1 1 6066999E
+P 13150 3650
+F 0 "#PWR0209" H 13150 3400 50  0001 C CNN
+F 1 "GND" H 13155 3477 50  0000 C CNN
+F 2 "" H 13150 3650 50  0001 C CNN
+F 3 "" H 13150 3650 50  0001 C CNN
+	1    13150 3650
+	1    0    0    -1
+$EndComp
+Text Label 13650 3850 2    50   ~ 0
+SSELC
+$Comp
+L Transistor_FET:2N7002 Q13
+U 1 1 606CC6F6
+P 13750 3650
+F 0 "Q13" V 13650 3550 50  0000 C CNN
+F 1 "2N7002" V 13650 3950 50  0000 C CNN
+F 2 "Package_TO_SOT_SMD:SOT-23" H 13950 3575 50  0001 L CIN
+F 3 "https://www.fairchildsemi.com/datasheets/2N/2N7002.pdf" H 13750 3650 50  0001 L CNN
+	1    13750 3650
+	0    -1   -1   0
+$EndComp
+$Comp
+L Device:R_Small R71
+U 1 1 606CC6FC
+P 13400 3550
+F 0 "R71" V 13300 3500 50  0000 L CNN
+F 1 "10K" V 13500 3450 50  0000 L CNN
+F 2 "Resistor_SMD:R_0805_2012Metric" H 13400 3550 50  0001 C CNN
+F 3 "~" H 13400 3550 50  0001 C CNN
+	1    13400 3550
+	0    -1   -1   0
+$EndComp
+Wire Wire Line
+	13500 3550 13550 3550
+$Comp
+L power:+12V #PWR0210
+U 1 1 606CC703
+P 13250 3500
+F 0 "#PWR0210" H 13250 3350 50  0001 C CNN
+F 1 "+12V" H 13265 3673 50  0000 C CNN
+F 2 "" H 13250 3500 50  0001 C CNN
+F 3 "" H 13250 3500 50  0001 C CNN
+	1    13250 3500
+	1    0    0    -1
+$EndComp
+Wire Wire Line
+	13650 3850 13750 3850
+Text Label 13700 3400 0    50   ~ 0
+SSELCH
+Wire Wire Line
+	14000 3650 14000 3550
+Wire Wire Line
+	14000 3550 13950 3550
+Connection ~ 13500 3550
+Wire Wire Line
+	13250 3500 13250 3550
+Wire Wire Line
+	13250 3550 13300 3550
+Wire Wire Line
+	13500 3400 13700 3400
+Wire Wire Line
+	13500 3400 13500 3550
+$Comp
+L power:GND #PWR0211
+U 1 1 606CC712
+P 14000 3650
+F 0 "#PWR0211" H 14000 3400 50  0001 C CNN
+F 1 "GND" H 14005 3477 50  0000 C CNN
+F 2 "" H 14000 3650 50  0001 C CNN
+F 3 "" H 14000 3650 50  0001 C CNN
+	1    14000 3650
+	1    0    0    -1
+$EndComp

Commit message: Stupid CH34G
Stupid CH34G
Parts:
- removed C10: 10uF, Capacitor_Tantalum_SMD:CP_EIA-6032-28_Kemet-C, symbol Device:CP_Small
- removed C21: 100nF, Capacitor_SMD:C_0805_2012Metric, symbol Device:C_Small
- added C10: 100nF, Capacitor_SMD:C_0805_2012Metric, symbol Device:C_Small
- added C21: 10uF, Capacitor_Tantalum_SMD:CP_EIA-6032-28_Kemet-C, symbol Device:CP_Small
Connections:
- net labels removed: VBUS
- wire segments 586 -> 580
- no-connect marks 12 -> 13
Changed lines of the file:
@@
 Wire Wire Line
 	14600 6050 14600 6100
-$Comp
-L power:VBUS #PWR0175
-U 1 1 600B49CF
-P 14600 4500
-F 0 "#PWR0175" H 14600 4350 50  0001 C CNN
-F 1 "VBUS" H 14615 4673 50  0000 C CNN
-F 2 "" H 14600 4500 50  0001 C CNN
-F 3 "" H 14600 4500 50  0001 C CNN
-	1    14600 4500
-	1    0    0    -1
-$EndComp
 Wire Wire Line
 	14600 4500 14600 4850
@@
 	15400 4550 15400 4500
 $Comp
-L power:VBUS #PWR0177
-U 1 1 609D5862
-P 15150 4500
-F 0 "#PWR0177" H 15150 4350 50  0001 C CNN
-F 1 "VBUS" H 15165 4673 50  0000 C CNN
-F 2 "" H 15150 4500 50  0001 C CNN
-F 3 "" H 15150 4500 50  0001 C CNN
-	1    15150 4500
-	1    0    0    -1
-$EndComp
-$Comp
-L power:VBUS #PWR0178
-U 1 1 609D5BF4
-P 15400 4500
-F 0 "#PWR0178" H 15400 4350 50  0001 C CNN
-F 1 "VBUS" H 15415 4673 50  0000 C CNN
-F 2 "" H 15400 4500 50  0001 C CNN
-F 3 "" H 15400 4500 50  0001 C CNN
-	1    15400 4500
-	1    0    0    -1
-$EndComp
-$Comp
 L Connector:USB_B_Mini J12
 U 1 1 609D7711
@@
 NoConn ~ 13450 5550
 $Comp
-L power:VBUS #PWR0179
-U 1 1 60ABEF15
-P 13500 4500
-F 0 "#PWR0179" H 13500 4350 50  0001 C CNN
-F 1 "VBUS" H 13515 4673 50  0000 C CNN
-F 2 "" H 13500 4500 50  0001 C CNN
-F 3 "" H 13500 4500 50  0001 C CNN
-	1    13500 4500
-	1    0    0    -1
-$EndComp
-Wire Wire Line
-	13500 4500 13500 4750
-Wire Wire Line
-	13500 5150 13450 5150
-$Comp
 L power:GND #PWR0180
 U 1 1 60B0DB32
@@
 Wire Wire Line
 	14200 5450 13450 5450
-$Comp
-L Device:CP_Small C10
-U 1 1 6112AB08
-P 13750 4900
-F 0 "C10" V 13838 4946 50  0000 L CNN
-F 1 "10uF" V 13600 4750 50  0000 L CNN
-F 2 "Capacitor_Tantalum_SMD:CP_EIA-6032-28_Kemet-C" H 13750 4900 50  0001 C CNN
-F 3 "~" H 13750 4900 50  0001 C CNN
-	1    13750 4900
-	1    0    0    -1
-$EndComp
-Wire Wire Line
-	13750 4800 13750 4750
-Wire Wire Line
-	13750 4750 13500 4750
-Connection ~ 13500 4750
-Wire Wire Line
-	13500 4750 13500 5150
-$Comp
-L power:GND #PWR0181
-U 1 1 6117C62D
-P 13750 5050
-F 0 "#PWR0181" H 13750 4800 50  0001 C CNN
-F 1 "GND" H 13755 4877 50  0000 C CNN
-F 2 "" H 13750 5050 50  0001 C CNN
-F 3 "" H 13750 5050 50  0001 C CNN
-	1    13750 5050
-	1    0    0    -1
-$EndComp
-Wire Wire Line
-	13750 5000 13750 5050
 Wire Notes Line
 	15800 4200 15800 6400
@@
 $EndComp
 $Comp
-L Device:C_Small C21
-U 1 1 605F6BC3
-P 15350 6000
-F 0 "C21" H 15442 6046 50  0000 L CNN
-F 1 "100nF" V 15550 5750 50  0000 L CNN
-F 2 "Capacitor_SMD:C_0805_2012Metric" H 15350 6000 50  0001 C CNN
-F 3 "~" H 15350 6000 50  0001 C CNN
-	1    15350 6000
-	1    0    0    -1
-$EndComp
-$Comp
-L power:GND #PWR0198
-U 1 1 605F6BCF
-P 15350 6100
-F 0 "#PWR0198" H 15350 5850 50  0001 C CNN
-F 1 "GND" H 15350 5950 50  0000 C CNN
-F 2 "" H 15350 6100 50  0001 C CNN
-F 3 "" H 15350 6100 50  0001 C CNN
-	1    15350 6100
-	1    0    0    -1
-$EndComp
-$Comp
-L power:VBUS #PWR0199
-U 1 1 6064EB08
-P 15350 5900
-F 0 "#PWR0199" H 15350 5750 50  0001 C CNN
-F 1 "VBUS" H 15365 6073 50  0000 C CNN
-F 2 "" H 15350 5900 50  0001 C CNN
-F 3 "" H 15350 5900 50  0001 C CNN
-	1    15350 5900
-	1    0    0    -1
-$EndComp
-$Comp
 L Device:C_Small C19
 U 1 1 60650E13
@@
 	1    0    0    -1
 $EndComp
+$Comp
+L power:+5V #PWR02
+U 1 1 601A4539
+P 14600 4500
+F 0 "#PWR02" H 14600 4350 50  0001 C CNN
+F 1 "+5V" H 14615 4673 50  0000 C CNN
+F 2 "" H 14600 4500 50  0001 C CNN
+F 3 "" H 14600 4500 50  0001 C CNN
+	1    14600 4500
+	1    0    0    -1
+$EndComp
+$Comp
+L power:+5V #PWR03
+U 1 1 601A4A43
+P 15150 4500
+F 0 "#PWR03" H 15150 4350 50  0001 C CNN
+F 1 "+5V" H 15165 4673 50  0000 C CNN
+F 2 "" H 15150 4500 50  0001 C CNN
+F 3 "" H 15150 4500 50  0001 C CNN
+	1    15150 4500
+	1    0    0    -1
+$EndComp
+$Comp
+L power:+5V #PWR04
+U 1 1 601A4C08
+P 15400 4500
+F 0 "#PWR04" H 15400 4350 50  0001 C CNN
+F 1 "+5V" H 15415 4673 50  0000 C CNN
+F 2 "" H 15400 4500 50  0001 C CNN
+F 3 "" H 15400 4500 50  0001 C CNN
+	1    15400 4500
+	1    0    0    -1
+$EndComp
+NoConn ~ 13450 5150
+$Comp
+L Device:C_Small C10
+U 1 1 6035A3FC
+P 15250 6000
+F 0 "C10" H 15300 5900 50  0000 L CNN
+F 1 "100nF" V 15100 5950 50  0000 L CNN
+F 2 "Capacitor_SMD:C_0805_2012Metric" H 15250 6000 50  0001 C CNN
+F 3 "~" H 15250 6000 50  0001 C CNN
+	1    15250 6000
+	1    0    0    -1
+$EndComp
+$Comp
+L power:GND #PWR05
+U 1 1 6035A402
+P 15250 6100
+F 0 "#PWR05" H 15250 5850 50  0001 C CNN
+F 1 "GND" H 15250 5950 50  0000 C CNN
+F 2 "" H 15250 6100 50  0001 C CNN
+F 3 "" H 15250 6100 50  0001 C CNN
+	1    15250 6100
+	1    0    0    -1
+$EndComp
+$Comp
+L power:+5V #PWR01
+U 1 1 603B6C27
+P 15250 5900
+F 0 "#PWR01" H 15250 5750 50  0001 C CNN
+F 1 "+5V" H 15265 6073 50  0000 C CNN
+F 2 "" H 15250 5900 50  0001 C CNN
+F 3 "" H 15250 5900 50  0001 C CNN
+	1    15250 5900
+	1    0    0    -1
+$EndComp
+$Comp
+L Device:CP_Small C21
+U 1 1 603CDAF6
+P 15650 6000
+F 0 "C21" V 15738 6046 50  0000 L CNN
+F 1 "10uF" V 15500 5850 50  0000 L CNN
+F 2 "Capacitor_Tantalum_SMD:CP_EIA-6032-28_Kemet-C" H 15650 6000 50  0001 C CNN
+F 3 "~" H 15650 6000 50  0001 C CNN
+	1    15650 6000
+	1    0    0    -1
+$EndComp
+$Comp
+L power:GND #PWR07
+U 1 1 603CDAFC
+P 15650 6100
+F 0 "#PWR07" H 15650 5850 50  0001 C CNN
+F 1 "GND" H 15650 5950 50  0000 C CNN
+F 2 "" H 15650 6100 50  0001 C CNN
+F 3 "" H 15650 6100 50  0001 C CNN
+	1    15650 6100
+	1    0    0    -1
+$EndComp
+$Comp
+L power:+5V #PWR06
+U 1 1 604E4FDF
+P 15650 5900
+F 0 "#PWR06" H 15650 5750 50  0001 C CNN
+F 1 "+5V" H 15665 6073 50  0000 C CNN
+F 2 "" H 15650 5900 50  0001 C CNN
+F 3 "" H 15650 5900 50  0001 C CNN
+	1    15650 5900
+	1    0    0    -1
+$EndComp

Commit message: Revert "Stupid CH34G"
This reverts commit 7f279e1c5784e09311cf2a8559607ba385112eda.
Parts:
- removed C10: 100nF, Capacitor_SMD:C_0805_2012Metric, symbol Device:C_Small
- removed C21: 10uF, Capacitor_Tantalum_SMD:CP_EIA-6032-28_Kemet-C, symbol Device:CP_Small
- added C10: 10uF, Capacitor_Tantalum_SMD:CP_EIA-6032-28_Kemet-C, symbol Device:CP_Small
- added C21: 100nF, Capacitor_SMD:C_0805_2012Metric, symbol Device:C_Small
Connections:
- net labels added: VBUS
- wire segments 580 -> 586
- no-connect marks 13 -> 12
Changed lines of the file:
@@
 Wire Wire Line
 	14600 6050 14600 6100
+$Comp
+L power:VBUS #PWR0175
+U 1 1 600B49CF
+P 14600 4500
+F 0 "#PWR0175" H 14600 4350 50  0001 C CNN
+F 1 "VBUS" H 14615 4673 50  0000 C CNN
+F 2 "" H 14600 4500 50  0001 C CNN
+F 3 "" H 14600 4500 50  0001 C CNN
+	1    14600 4500
+	1    0    0    -1
+$EndComp
 Wire Wire Line
 	14600 4500 14600 4850
@@
 	15400 4550 15400 4500
 $Comp
+L power:VBUS #PWR0177
+U 1 1 609D5862
+P 15150 4500
+F 0 "#PWR0177" H 15150 4350 50  0001 C CNN
+F 1 "VBUS" H 15165 4673 50  0000 C CNN
+F 2 "" H 15150 4500 50  0001 C CNN
+F 3 "" H 15150 4500 50  0001 C CNN
+	1    15150 4500
+	1    0    0    -1
+$EndComp
+$Comp
+L power:VBUS #PWR0178
+U 1 1 609D5BF4
+P 15400 4500
+F 0 "#PWR0178" H 15400 4350 50  0001 C CNN
+F 1 "VBUS" H 15415 4673 50  0000 C CNN
+F 2 "" H 15400 4500 50  0001 C CNN
+F 3 "" H 15400 4500 50  0001 C CNN
+	1    15400 4500
+	1    0    0    -1
+$EndComp
+$Comp
 L Connector:USB_B_Mini J12
 U 1 1 609D7711
@@
 NoConn ~ 13450 5550
 $Comp
+L power:VBUS #PWR0179
+U 1 1 60ABEF15
+P 13500 4500
+F 0 "#PWR0179" H 13500 4350 50  0001 C CNN
+F 1 "VBUS" H 13515 4673 50  0000 C CNN
+F 2 "" H 13500 4500 50  0001 C CNN
+F 3 "" H 13500 4500 50  0001 C CNN
+	1    13500 4500
+	1    0    0    -1
+$EndComp
+Wire Wire Line
+	13500 4500 13500 4750
+Wire Wire Line
+	13500 5150 13450 5150
+$Comp
 L power:GND #PWR0180
 U 1 1 60B0DB32
@@
 Wire Wire Line
 	14200 5450 13450 5450
+$Comp
+L Device:CP_Small C10
+U 1 1 6112AB08
+P 13750 4900
+F 0 "C10" V 13838 4946 50  0000 L CNN
+F 1 "10uF" V 13600 4750 50  0000 L CNN
+F 2 "Capacitor_Tantalum_SMD:CP_EIA-6032-28_Kemet-C" H 13750 4900 50  0001 C CNN
+F 3 "~" H 13750 4900 50  0001 C CNN
+	1    13750 4900
+	1    0    0    -1
+$EndComp
+Wire Wire Line
+	13750 4800 13750 4750
+Wire Wire Line
+	13750 4750 13500 4750
+Connection ~ 13500 4750
+Wire Wire Line
+	13500 4750 13500 5150
+$Comp
+L power:GND #PWR0181
+U 1 1 6117C62D
+P 13750 5050
+F 0 "#PWR0181" H 13750 4800 50  0001 C CNN
+F 1 "GND" H 13755 4877 50  0000 C CNN
+F 2 "" H 13750 5050 50  0001 C CNN
+F 3 "" H 13750 5050 50  0001 C CNN
+	1    13750 5050
+	1    0    0    -1
+$EndComp
+Wire Wire Line
+	13750 5000 13750 5050
 Wire Notes Line
 	15800 4200 15800 6400
@@
 $EndComp
 $Comp
+L Device:C_Small C21
+U 1 1 605F6BC3
+P 15350 6000
+F 0 "C21" H 15442 6046 50  0000 L CNN
+F 1 "100nF" V 15550 5750 50  0000 L CNN
+F 2 "Capacitor_SMD:C_0805_2012Metric" H 15350 6000 50  0001 C CNN
+F 3 "~" H 15350 6000 50  0001 C CNN
+	1    15350 6000
+	1    0    0    -1
+$EndComp
+$Comp
+L power:GND #PWR0198
+U 1 1 605F6BCF
+P 15350 6100
+F 0 "#PWR0198" H 15350 5850 50  0001 C CNN
+F 1 "GND" H 15350 5950 50  0000 C CNN
+F 2 "" H 15350 6100 50  0001 C CNN
+F 3 "" H 15350 6100 50  0001 C CNN
+	1    15350 6100
+	1    0    0    -1
+$EndComp
+$Comp
+L power:VBUS #PWR0199
+U 1 1 6064EB08
+P 15350 5900
+F 0 "#PWR0199" H 15350 5750 50  0001 C CNN
+F 1 "VBUS" H 15365 6073 50  0000 C CNN
+F 2 "" H 15350 5900 50  0001 C CNN
+F 3 "" H 15350 5900 50  0001 C CNN
+	1    15350 5900
+	1    0    0    -1
+$EndComp
+$Comp
 L Device:C_Small C19
 U 1 1 60650E13
@@
 	1    0    0    -1
 $EndComp
-$Comp
-L power:+5V #PWR02
-U 1 1 601A4539
-P 14600 4500
-F 0 "#PWR02" H 14600 4350 50  0001 C CNN
-F 1 "+5V" H 14615 4673 50  0000 C CNN
-F 2 "" H 14600 4500 50  0001 C CNN
-F 3 "" H 14600 4500 50  0001 C CNN
-	1    14600 4500
-	1    0    0    -1
-$EndComp
-$Comp
-L power:+5V #PWR03
-U 1 1 601A4A43
-P 15150 4500
-F 0 "#PWR03" H 15150 4350 50  0001 C CNN
-F 1 "+5V" H 15165 4673 50  0000 C CNN
-F 2 "" H 15150 4500 50  0001 C CNN
-F 3 "" H 15150 4500 50  0001 C CNN
-	1    15150 4500
-	1    0    0    -1
-$EndComp
-$Comp
-L power:+5V #PWR04
-U 1 1 601A4C08
-P 15400 4500
-F 0 "#PWR04" H 15400 4350 50  0001 C CNN
-F 1 "+5V" H 15415 4673 50  0000 C CNN
-F 2 "" H 15400 4500 50  0001 C CNN
-F 3 "" H 15400 4500 50  0001 C CNN
-	1    15400 4500
-	1    0    0    -1
-$EndComp
-NoConn ~ 13450 5150
-$Comp
-L Device:C_Small C10
-U 1 1 6035A3FC
-P 15250 6000
-F 0 "C10" H 15300 5900 50  0000 L CNN
-F 1 "100nF" V 15100 5950 50  0000 L CNN
-F 2 "Capacitor_SMD:C_0805_2012Metric" H 15250 6000 50  0001 C CNN
-F 3 "~" H 15250 6000 50  0001 C CNN
-	1    15250 6000
-	1    0    0    -1
-$EndComp
-$Comp
-L power:GND #PWR05
-U 1 1 6035A402
-P 15250 6100
-F 0 "#PWR05" H 15250 5850 50  0001 C CNN
-F 1 "GND" H 15250 5950 50  0000 C CNN
-F 2 "" H 15250 6100 50  0001 C CNN
-F 3 "" H 15250 6100 50  0001 C CNN
-	1    15250 6100
-	1    0    0    -1
-$EndComp
-$Comp
-L power:+5V #PWR01
-U 1 1 603B6C27
-P 15250 5900
-F 0 "#PWR01" H 15250 5750 50  0001 C CNN
-F 1 "+5V" H 15265 6073 50  0000 C CNN
-F 2 "" H 15250 5900 50  0001 C CNN
-F 3 "" H 15250 5900 50  0001 C CNN
-	1    15250 5900
-	1    0    0    -1
-$EndComp
-$Comp
-L Device:CP_Small C21
-U 1 1 603CDAF6
-P 15650 6000
-F 0 "C21" V 15738 6046 50  0000 L CNN
-F 1 "10uF" V 15500 5850 50  0000 L CNN
-F 2 "Capacitor_Tantalum_SMD:CP_EIA-6032-28_Kemet-C" H 15650 6000 50  0001 C CNN
-F 3 "~" H 15650 6000 50  0001 C CNN
-	1    15650 6000
-	1    0    0    -1
-$EndComp
-$Comp
-L power:GND #PWR07
-U 1 1 603CDAFC
-P 15650 6100
-F 0 "#PWR07" H 15650 5850 50  0001 C CNN
-F 1 "GND" H 15650 5950 50  0000 C CNN
-F 2 "" H 15650 6100 50  0001 C CNN
-F 3 "" H 15650 6100 50  0001 C CNN
-	1    15650 6100
-	1    0    0    -1
-$EndComp
-$Comp
-L power:+5V #PWR06
-U 1 1 604E4FDF
-P 15650 5900
-F 0 "#PWR06" H 15650 5750 50  0001 C CNN
-F 1 "+5V" H 15665 6073 50  0000 C CNN
-F 2 "" H 15650 5900 50  0001 C CNN
-F 3 "" H 15650 5900 50  0001 C CNN
-	1    15650 5900
-	1    0    0    -1
-$EndComp

Commit message: Kicad is silly
Parts:
- J12: symbol Connector:USB_B_Mini -> cnc-universal-input-rescue:USB_B_Mini-Connector
Changed lines of the file:
@@
 $EndComp
 $Comp
-L Connector:USB_B_Mini J12
+L cnc-universal-input-rescue:USB_B_Mini-Connector J12
 U 1 1 609D7711
 P 13150 5350
